File: LEDLightHardware.sch (KiCad schematic (older format))
At the start: 7 parts

Commit message: Reorganized
Parts:
- removed C?: 22u, symbol C
- removed C?: 10u, symbol C
- removed U?: LM7805CT, TO-220, symbol LM7805CT
- added C2: 22u, Capacitors_ThroughHole:C_Radial_D5_L11_P2.5, symbol CP
- added C3: 10u, Capacitors_ThroughHole:C_Radial_D5_L11_P2.5, symbol CP
- added U1: LM7805(Has_numbers), Power_Integrations:TO-220, symbol LM7805(Has_numbers)
- C1: renamed from C?; footprint (none) -> Capacitors_ThroughHole:C_Disc_D6_P5
- IC1: renamed from IC?; footprint DIP8 -> Housings_DIP:DIP-8_W7.62mm_LongPads
- P1, P2: renamed from P?; footprint (none) -> Pin_Headers:Pin_Header_Straight_1x03
Changed lines of the file:
@@
 LIBS:contrib
 LIBS:valves
+LIBS:TedsComponents
 LIBS:LEDLightHardware-cache
 EELAYER 25 0
@@
 $Descr A4 11693 8268
 encoding utf-8
-Sheet 1 1
+Sheet 1 2
 Title ""
 Date ""
@@
 $EndDescr
 $Comp
-L ATTINY45-P IC?
+L ATTINY45-P IC1
 U 1 1 56FFFE4D
 P 2700 1450
-F 0 "IC?" H 1550 1850 50  0000 C CNN
+F 0 "IC1" H 1550 1850 50  0000 C CNN
 F 1 "ATTINY45-P" H 3700 1050 50  0000 C CNN
-F 2 "DIP8" H 3700 1450 50  0000 C CIN
+F 2 "Housings_DIP:DIP-8_W7.62mm_LongPads" H 3700 1450 50  0000 C CIN
 F 3 "" H 2700 1450 50  0000 C CNN
 	1    2700 1450
@@
 	1250 1200 1350 1200
 $Comp
-L GND #PWR?
+L GND #PWR2
 U 1 1 56FFFF6F
 P 1250 1750
-F 0 "#PWR?" H 1250 1500 50  0001 C CNN
+F 0 "#PWR2" H 1250 1500 50  0001 C CNN
 F 1 "GND" H 1250 1600 50  0000 C CNN
 F 2 "" H 1250 1750 50  0000 C CNN
@@
 NoConn ~ 4050 1600
 $Comp
-L VCC #PWR?
+L VCC #PWR3
 U 1 1 57012428
 P 1650 2700
-F 0 "#PWR?" H 1650 2550 50  0001 C CNN
+F 0 "#PWR3" H 1650 2550 50  0001 C CNN
 F 1 "VCC" H 1650 2850 50  0000 C CNN
 F 2 "" H 1650 2700 50  0000 C CNN
@@
 	1650 2750 1800 2750
 $Comp
-L GND #PWR?
+L GND #PWR4
 U 1 1 5701244A
 P 1650 2900
-F 0 "#PWR?" H 1650 2650 50  0001 C CNN
+F 0 "#PWR4" H 1650 2650 50  0001 C CNN
 F 1 "GND" H 1650 2750 50  0000 C CNN
 F 2 "" H 1650 2900 50  0000 C CNN
@@
 	1650 2850 1800 2850
 $Comp
-L C C?
+L C C1
 U 1 1 570124BC
 P 1250 1450
-F 0 "C?" H 1275 1550 50  0000 L CNN
+F 0 "C1" H 1275 1550 50  0000 L CNN
 F 1 "u10" H 1275 1350 50  0000 L CNN
-F 2 "" H 1288 1300 50  0000 C CNN
+F 2 "Capacitors_ThroughHole:C_Disc_D6_P5" H 1288 1300 50  0001 C CNN
 F 3 "" H 1250 1450 50  0000 C CNN
 	1    1250 1450
@@
 Vcc = 12V
 $Comp
-L LM7805CT U?
-U 1 1 57012653
-P 3900 2650
-F 0 "U?" H 3700 2850 50  0000 C CNN
-F 1 "LM7805CT" H 3900 2850 50  0000 L CNN
-F 2 "TO-220" H 3900 2750 50  0000 C CIN
-F 3 "" H 3900 2650 50  0000 C CNN
-	1    3900 2650
-	1    0    0    -1
-$EndComp
-$Comp
-L VCC #PWR?
+L VCC #PWR5
 U 1 1 570126D6
 P 3350 2550
-F 0 "#PWR?" H 3350 2400 50  0001 C CNN
+F 0 "#PWR5" H 3350 2400 50  0001 C CNN
 F 1 "VCC" H 3350 2700 50  0000 C CNN
 F 2 "" H 3350 2550 50  0000 C CNN
@@
 	3900 2900 3900 3150
 $Comp
-L +5V #PWR?
+L +5V #PWR7
 U 1 1 57012788
 P 4550 2550
-F 0 "#PWR?" H 4550 2400 50  0001 C CNN
+F 0 "#PWR7" H 4550 2400 50  0001 C CNN
 F 1 "+5V" H 4550 2690 50  0000 C CNN
 F 2 "" H 4550 2550 50  0000 C CNN
@@
 	4550 2600 4300 2600
 $Comp
-L +5V #PWR?
+L +5V #PWR1
 U 1 1 5701281E
 P 1250 1050
-F 0 "#PWR?" H 1250 900 50  0001 C CNN
+F 0 "#PWR1" H 1250 900 50  0001 C CNN
 F 1 "+5V" H 1250 1190 50  0000 C CNN
 F 2 "" H 1250 1050 50  0000 C CNN
@@
 	1    0    0    -1
 $EndComp
-$Comp
-L C C?
-U 1 1 570129AF
-P 3400 2850
-F 0 "C?" H 3425 2950 50  0000 L CNN
-F 1 "22u" H 3425 2750 50  0000 L CNN
-F 2 "" H 3438 2700 50  0000 C CNN
-F 3 "" H 3400 2850 50  0000 C CNN
-	1    3400 2850
-	1    0    0    -1
-$EndComp
 Wire Wire Line
 	3400 3000 3400 3050
@@
 	3400 3050 4450 3050
 $Comp
-L GND #PWR?
+L GND #PWR6
 U 1 1 57012A19
 P 3900 3150
-F 0 "#PWR?" H 3900 2900 50  0001 C CNN
+F 0 "#PWR6" H 3900 2900 50  0001 C CNN
 F 1 "GND" H 3900 3000 50  0000 C CNN
 F 2 "" H 3900 3150 50  0000 C CNN
@@
 $EndComp
 Connection ~ 3900 3050
-$Comp
-L C C?
-U 1 1 57012A54
-P 4450 2850
-F 0 "C?" H 4475 2950 50  0000 L CNN
-F 1 "10u" H 4475 2750 50  0000 L CNN
-F 2 "" H 4488 2700 50  0000 C CNN
-F 3 "" H 4450 2850 50  0000 C CNN
-	1    4450 2850
-	1    0    0    -1
-$EndComp
 Wire Wire Line
 	4450 3050 4450 3000
@@
 Connection ~ 3400 2600
 $Comp
-L CONN_01X03 P?
+L CONN_01X03 P2
 U 1 1 57012C0D
 P 5600 2100
-F 0 "P?" H 5600 2300 50  0000 C CNN
+F 0 "P2" H 5600 2300 50  0000 C CNN
 F 1 "CONN_01X03" V 5700 2100 50  0000 C CNN
-F 2 "" H 5600 2100 50  0000 C CNN
+F 2 "Pin_Headers:Pin_Header_Straight_1x03" H 5600 2100 50  0001 C CNN
 F 3 "" H 5600 2100 50  0000 C CNN
 	1    5600 2100
@@
 $EndComp
 $Comp
-L VCC #PWR?
+L VCC #PWR9
 U 1 1 57012CFB
 P 5250 1950
-F 0 "#PWR?" H 5250 1800 50  0001 C CNN
+F 0 "#PWR9" H 5250 1800 50  0001 C CNN
 F 1 "VCC" H 5250 2100 50  0000 C CNN
 F 2 "" H 5250 1950 50  0000 C CNN
@@
 	5250 2000 5400 2000
 $Comp
-L GND #PWR?
+L GND #PWR8
 U 1 1 57012D3F
 P 5150 2100
-F 0 "#PWR?" H 5150 1850 50  0001 C CNN
+F 0 "#PWR8" H 5150 1850 50  0001 C CNN
 F 1 "GND" H 5150 1950 50  0000 C CNN
 F 2 "" H 5150 2100 50  0000 C CNN
@@
 	5400 2350 5400 2200
 $Comp
-L CONN_01X03 P?
+L CONN_01X03 P1
 U 1 1 5701301E
 P 2000 2850
-F 0 "P?" H 2000 3050 50  0000 C CNN
+F 0 "P1" H 2000 3050 50  0000 C CNN
 F 1 "CONN_01X03" V 2100 2850 50  0000 C CNN
-F 2 "" H 2000 2850 50  0000 C CNN
+F 2 "Pin_Headers:Pin_Header_Straight_1x03" H 2000 2850 50  0001 C CNN
 F 3 "" H 2000 2850 50  0000 C CNN
 	1    2000 2850
@@
 Wire Wire Line
 	1750 2950 1800 2950
+$Comp
+L CP C2
+U 1 1 57012D29
+P 3400 2850
+F 0 "C2" H 3425 2950 50  0000 L CNN
+F 1 "22u" H 3425 2750 50  0000 L CNN
+F 2 "Capacitors_ThroughHole:C_Radial_D5_L11_P2.5" H 3438 2700 50  0001 C CNN
+F 3 "" H 3400 2850 50  0000 C CNN
+	1    3400 2850
+	1    0    0    -1
+$EndComp
+$Comp
+L CP C3
+U 1 1 57012DDB
+P 4450 2850
+F 0 "C3" H 4475 2950 50  0000 L CNN
+F 1 "10u" H 4475 2750 50  0000 L CNN
+F 2 "Capacitors_ThroughHole:C_Radial_D5_L11_P2.5" H 4488 2700 50  0001 C CNN
+F 3 "" H 4450 2850 50  0000 C CNN
+	1    4450 2850
+	1    0    0    -1
+$EndComp
+$Comp
+L LM7805(Has_numbers) U1
+U 1 1 57012ED7
+P 3900 2650
+F 0 "U1" H 4050 2454 60  0000 C CNN
+F 1 "LM7805(Has_numbers)" H 3900 2850 60  0000 C CNN
+F 2 "Power_Integrations:TO-220" H 3900 2650 60  0001 C CNN
+F 3 "" H 3900 2650 60  0000 C CNN
+	1    3900 2650
+	1    0    0    -1
+$EndComp
+$Sheet
+S 1400 4300 2000 1400
+U 570176C3
+F0 "8266Section" 60
+F1 "file570176C2.sch" 60
+$EndSheet
 $EndSCHEMATC
